File: Controller PCB/Water Auto Turret Main Board.sch (EAGLE design)
At the start: 39 parts, among them IC1 DRV8806PWP, IC2 L7805ACV, IC3 PIC12F683-I_P, IC4 SN74LVC2G08DCTR, J1 78171-0004, J10 47053-1000, J2 7691, J3 7691, J4 47053-1000, J5 47053-1000, J6 47053-1000, J7 47053-1000, J8 47053-1000, J9 47053-1000, K1 G5RL-K1A-E, Q1 BC33716BU, Q2 BC33716BU

Commit message: Rev2 PCB
Fixes issues found on Rev1 PCB
Parts:
- removed C7: C322C104K1R5TA, SamacSys_Parts:C322C104K1R5TA
- removed IC4: SN74LVC2G08DCTR, SamacSys_Parts:SN74LVC2G08DCTR
- added C4: C322C104K1R5TA, SamacSys_Parts:C322C104K1R5TA
- added JP4: (no value), pinhead:PINHD-1X3
- added R10, R11, R8, R9: 8k, resistor:R-EU_V234/12
- added R5: 1k37, resistor:R-EU_V234/12
- C2: value 16SEPC100M+TSS -> C322C104K1R5TA; device SamacSys_Parts:16SEPC100M+TSS -> SamacSys_Parts:C322C104K1R5TA
- C5: value C322C104K1R5TA -> 16SEPC100M+TSS; device SamacSys_Parts:C322C104K1R5TA -> SamacSys_Parts:16SEPC100M+TSS
- IC1: value DRV8806PWP -> L7805ACV; device SamacSys_Parts:DRV8806PWP -> SamacSys_Parts:L7805ACV
- IC2: value L7805ACV -> PIC12F683-I_P; device SamacSys_Parts:L7805ACV -> SamacSys_Parts:PIC12F675-I_P
- IC3: value PIC12F683-I_P -> DRV8806PWP; device SamacSys_Parts:PIC12F675-I_P -> SamacSys_Parts:DRV8806PWP
- J1: value 78171-0004 -> 7691; device SamacSys_Parts:78171-0004 -> SamacSys_Parts-old:7691
- J11: value (none) -> 47053-1000; device VIM3GPIO:VIM3GPIO -> SamacSys_Parts-old:47053-1000
- J3: value 7691 -> 47053-1000; device SamacSys_Parts-old:7691 -> SamacSys_Parts-old:47053-1000
- J4: value 47053-1000 -> 78171-0004; device SamacSys_Parts-old:47053-1000 -> SamacSys_Parts:78171-0004
- J5: MANUFACTURER_PART_NUMBER (none) -> Solenoid 1 & 2
- J6: MANUFACTURER_PART_NUMBER Solenoid 1 & 2 -> (none)
- J7: value 47053-1000 -> (none); device SamacSys_Parts-old:47053-1000 -> VIM3GPIO:VIM3GPIO
- JP2: value (none) -> Fan Header
- JP3: device pinhead:PINHD-1X3 -> pinhead:PINHD-1X2
- R1: value 8k -> 1k
- R2: value 3k6 -> 1k
- R3: value 1k -> 8k; device resistor:R-EU_V234/12 -> resistor:R-EU_0309/V
- R4: value 1k -> 1k37
- R6: value (none) -> 8k
- R7: value (none) -> 3k6; device resistor:R-EU_V234/12 -> resistor:R-EU_0309/V
Connections:
- removed net N$34: IC4.1Y, U1.CSN
- removed net N$41: IC4.VCC, J11.3V3_2, U1.VCC_IO
- removed net N$46: J11.3V3_1, U2.VCC_IO
- net +12V: now also C2.1, C4.1, C5.+, IC1.INPUT, IC3.VCLAMP, IC3.VM, J1.3, J1.4, J4.1, J4.2, J5.1, J5.3, JP2.1, R6.1; no longer C2.+, C5.1, C7.1, IC1.VCLAMP, IC1.VM, IC2.INPUT, J2.1, J2.2, J2.3, J2.4, J7.1, J7.3, R1.1
- net +5V: now also D3.K, IC1.OUTPUT, IC2.VDD, J3.3, R3.1; no longer D4.K, IC2.OUTPUT, IC3.VDD, J10.3
- net GND: now also D4.A, IC1.GND, IC2.VSS, J2.1, J2.2, J2.3, J2.4, JP2.2, R7.2; no longer D3.A, IC2.GND, IC3.VSS, J3.1, J3.2, J3.3, J3.4, R2.2
- net N$1: now also IC3.OUT2, J5.2; no longer IC1.OUT2, J6.2
- net N$10: now also R4.1; no longer R6.1
- net N$11: now also IC2.GP0/AN0/CIN+/ICSPDAT, R2.2; no longer IC3.GP0/AN0/CIN+/ICSPDAT, R4.2
- net N$12: now also IC2.GP1/AN1/CIN-/VREF/ICSPCLK, JP3.2; no longer IC3.GP1/AN1/CIN-/VREF/ICSPCLK, JP2.2
- net N$13: now also R5.1; no longer R7.1
- net N$14: now also IC2.GP4/AN3/!T1G!/OSC2/CLKOUT, R5.2; no longer IC3.GP4/AN3/!T1G!/OSC2/CLKOUT, R7.2
- net N$15: now also IC2.GP5/T1CKI/OSC1/CLKIN, R4.2; no longer IC3.GP5/T1CKI/OSC1/CLKIN, R6.2
- net N$16: now also D3.A, D4.K, IC2.GP2/AN2/T0CKI/INT/COUT, R6.2, R7.1; no longer D3.K, D4.A, IC3.GP2/AN2/T0CKI/INT/COUT, R1.2, R2.1
- net N$17: now also J3.4, JP3.1, R3.2; no longer J10.4, JP2.1
- net N$18: now also J7.PWM_F; no longer J11.PWM_F
- net N$19: now also J7.GPIOH_4; no longer J11.GPIOH_4
- net N$2: now also IC3.OUT1, J5.4; no longer IC1.OUT1, J6.4
- net N$20: now also J7.UARTC_TX; no longer J11.UARTC_TX
- net N$21: now also J10.4; no longer J4.4
- net N$22: now also J10.3; no longer J4.3
- net N$23: now also J10.1; no longer J4.1
- net N$24: now also J10.2; no longer J4.2
- net N$25: now also J11.4; no longer J5.4
- net N$26: now also J11.2; no longer J5.2
- net N$27: now also J11.1; no longer J5.1
- net N$28: now also J11.3; no longer J5.3
- net N$29: now also R9.2
- net N$3: now also IC3.OUT3, J6.4; no longer IC1.OUT3, J7.4
- net N$30: now also R8.2
- net N$31: now also R11.2
- net N$32: now also R10.2
- net N$33: now also J7.3V3_1, R10.1, R11.1, U2.VCC_IO; no longer IC4.1A, IC4.2A, J11.UARTC_RX
- net N$35: now also IC3.SDATIN, J7.I2SB_SCLK; no longer IC1.SDATIN, J11.I2SB_SCLK
- net N$36: now also IC3.SCLK, J7.I2SB_SDO; no longer IC1.SCLK, J11.I2SB_SDO
- net N$37: now also IC3.LATCH, J7.I2SB_LRCK; no longer IC1.LATCH, J11.I2SB_LRCK
- net N$38: now also IC3.RESET, J7.I2SB_SDI; no longer IC1.RESET, J11.I2SB_SDI
- net N$39: now also J7.LINUX_RX, JP4.3; no longer J11.LINUX_RX, JP3.3
- net N$4: now also IC3.OUT4, J6.2; no longer IC1.OUT4, J7.2
- net N$40: now also J7.LINUX_TX, JP4.2; no longer J11.LINUX_TX, JP3.2
- net N$42: now also J7.3V3_2, R8.1, R9.1, U1.VCC_IO; no longer IC4.2Y, U2.CSN
- net N$44: now also J7.I2C_M3_SCL, U1.CSN; no longer IC4.1B, J11.I2C_M3_SCL
- net N$45: now also J7.I2C_M3_SDA, U2.CSN; no longer IC4.2B, J11.I2C_M3_SDA
- net N$5: now also J3.1, R1.2; no longer J10.1, R3.2
- net N$8: now also J3.2, R2.1; no longer J10.2, R4.1
- net N$9: now also IC2.GP3/!MCLR!/VPP; no longer IC3.GP3/!MCLR!/VPP
- net VSS: now also C2.2, C4.2, C5.-, IC3.GND_1, IC3.GND_2, IC3.GND_3, IC3.NENBL, J4.3, J4.4, J7.GND@1, J7.GND@2, J7.GND@3, J7.GND@4, J7.GND@5, J7.GND@6, J7.GND@7, J7.GND@8, J7.GND@9, JP4.1, R1.1; no longer C2.-, C5.2, C7.2, IC1.GND_1, IC1.GND_2, IC1.GND_3, IC1.NENBL, IC4.GND, J1.3, J1.4, J11.GND@1, J11.GND@2, J11.GND@3, J11.GND@4, J11.GND@5, J11.GND@6, J11.GND@7, J11.GND@8, J11.GND@9, JP3.1, R3.1
Other:
- moved on the sheet: C3, C6, D3, D4, J10, J2, J3, J5, J6, JP2, R1, R2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
